Commit message: feat: add color to the robot

File: src/my_robot/urdf/my_robot.xacro (robot description, xacro)
@@ -2,4 +2,13 @@
 <robot name="my_robot" xmlns:xacro="http://www.ros.org/wiki/xacro">
   <xacro:include filename="$(find my_robot)/urdf/my_robot.gazebo"/>
+  <material name="orange">
+    <color rgba="1 0.64 0 1"/>
+  </material>
+  <material name="white">
+    <color rgba="1 1 1 1"/>
+  </material>
+  <material name="black">
+    <color rgba="0 0 0 1"/>
+  </material>
   <link name="robot_footprint"></link>
   <joint name="robot_footprint_joint" type="fixed">
@@ -30,4 +39,5 @@
         <box size=".4 .2 .1"/>
       </geometry>
+      <material name="black"/>
     </visual>
     <collision name='back_caster_collision'>
@@ -42,4 +52,5 @@
         <sphere radius="0.05"/>
       </geometry>
+      <material name="orange"/>
     </visual>
     <collision name='front_caster_collision'>
@@ -54,4 +65,5 @@
         <sphere radius="0.05"/>
       </geometry>
+      <material name="white"/>
     </visual>
   </link>
@@ -77,4 +89,5 @@
         <cylinder radius="0.1" length="0.05"/>
       </geometry>
+      <material name="orange"/>
     </visual>
   </link>
@@ -100,4 +113,5 @@
         <cylinder radius="0.1" length="0.05"/>
       </geometry>
+      <material name="orange"/>
     </visual>
   </link>
@@ -139,4 +153,5 @@
         <box size=".05 .05 .05"/>
       </geometry>
+      <material name="white"/>
     </visual>
   </link>

Commit message: change robot model color in gazebo and rviz

File: src/my_robot/urdf/my_robot.xacro (robot description, xacro)
@@ -11,4 +11,7 @@
     <color rgba="0 0 0 1"/>
   </material>
+  <material name="green">
+    <color rgba="0 1 0 1"/>
+  </material>
   <link name="robot_footprint"></link>
   <joint name="robot_footprint_joint" type="fixed">
@@ -17,4 +20,7 @@
     <child link="chassis" />
   </joint>
+  <gazebo reference='chassis'>
+    <material>Gazebo/Black</material>
+  </gazebo>
   <link name='chassis'>
     <pose>0 0 0.1 0 0 0</pose>
@@ -36,8 +42,8 @@
     <visual name='chassis_visual'>
       <origin xyz="0 0 0" rpy=" 0 0 0"/>
+      <material name="black"/>
       <geometry>
         <box size=".4 .2 .1"/>
       </geometry>
-      <material name="black"/>
     </visual>
     <collision name='back_caster_collision'>
@@ -68,5 +74,8 @@
     </visual>
   </link>
-  <link name="right_wheel">
+  <gazebo reference='right_wheel'>
+    <material>Gazebo/Orange</material>
+  </gazebo>
+  <link name='right_wheel'>
     <inertial>
       <mass value="5"/>
@@ -78,11 +87,11 @@
         />
     </inertial>
-    <collision name="righ_wheel_collision">
-      <origin xyz="0 0 0" rpy="0 1.5707 1.5707"/>
-      <geometry>
-        <cylinder radius="0.1" length="0.05"/>
-      </geometry>
-    </collision>
-    <visual name="righ_wheel_visual">
+    <collision name="right_wheel_collision">
+      <origin xyz="0 0 0" rpy="0 1.5707 1.5707"/>
+      <geometry>
+        <cylinder radius="0.1" length="0.05"/>
+      </geometry>
+    </collision>
+    <visual name="right_wheel_visual">
       <origin xyz="0 0 0" rpy="0 1.5707 1.5707"/>
       <geometry>
@@ -92,5 +101,8 @@
     </visual>
   </link>
-  <link name="left_wheel">
+  <gazebo reference='left_wheel'>
+    <material>Gazebo/Orange</material>
+  </gazebo>
+  <link name='left_wheel'>
     <inertial>
       <mass value="5"/>
@@ -102,11 +114,11 @@
         />
     </inertial>
-    <collision name="righ_wheel_collision">
-      <origin xyz="0 0 0" rpy="0 1.5707 1.5707"/>
-      <geometry>
-        <cylinder radius="0.1" length="0.05"/>
-      </geometry>
-    </collision>
-    <visual name="righ_wheel_visual">
+    <collision name="left_wheel_collision">
+      <origin xyz="0 0 0" rpy="0 1.5707 1.5707"/>
+      <geometry>
+        <cylinder radius="0.1" length="0.05"/>
+      </geometry>
+    </collision>
+    <visual name="left_wheel_visual">
       <origin xyz="0 0 0" rpy="0 1.5707 1.5707"/>
       <geometry>
@@ -132,4 +144,7 @@
     <dynamics damping="1.0" friction="1.0"/>
   </joint>
+  <gazebo reference='camera'>
+    <material>Gazebo/Green</material>
+  </gazebo>
   <link name="camera">
     <inertial>
@@ -153,5 +168,5 @@
         <box size=".05 .05 .05"/>
       </geometry>
-      <material name="white"/>
+      <material name="green"/>
     </visual>
   </link>
